File: terminal-variant-pcb/kicad/water-level-pressure.kicad_pcb (KiCad board)
At the start: 2 copper layers, 93.3 x 60.1 mm, 38 parts, among them J1 Conn_01x03, J3 Conn_01x02, T1 TestPoint, T10 TestPoint, T11 TestPoint, T12 TestPoint, T13 TestPoint, T14 TestPoint, T15 TestPoint, T16 TestPoint, T17 TestPoint, T18 TestPoint, T19 TestPoint, T2 TestPoint, T20 TestPoint, T21 TestPoint, T22 TestPoint, T23 TestPoint, T24 TestPoint, T25 TestPoint, T26 TestPoint, T27 TestPoint, T28 TestPoint, T29 TestPoint, T3 TestPoint, T30 TestPoint, T4 TestPoint, T5 TestPoint, T6 TestPoint, T7 TestPoint, T8 TestPoint, T9 TestPoint

Commit message: Add LCD connector. First draft. Update PDF schematic. Remove old SVG schematic.
Parts:
- added J2: Conn_01x04, Connector_PinHeader_2.54mm:PinHeader_1x04_P2.54mm_Vertical_SMD_Pin1Left, F.Cu at (204.6, 99.7)
Connections:
- net Net-(A1-SCL/A5) renamed /SCL
- net Net-(A1-SDA/A4) renamed /SDA
Routing:
- net /SCL: track 3.56 -> 80.6 mm
- net /SDA: track 3.56 -> 76.1 mm
- net +5V: track 74.5 -> 120.0 mm, vias 0 -> 6
- net GND: track 3.56 -> 13.2 mm
- net /LEVEL: track 94.1 -> 96.5 mm, vias 0 -> 4
Other:
- board text added: "LCD"
- board text added: "SCL"
- board text added: "SDA"
