File: terminal-variant-pcb/kicad/water-level-pressure.kicad_pcb (KiCad board)
At the start: 2 copper layers, 93.3 x 60.1 mm, 40 parts, among them J1 Conn_01x03, J2 Conn_01x04, J3 Conn_01x02, J4 Conn_01x15_Socket, J5 Conn_01x15_Socket, T1 TestPoint, T10 TestPoint, T11 TestPoint, T12 TestPoint, T13 TestPoint, T14 TestPoint, T15 TestPoint, T16 TestPoint, T17 TestPoint, T18 TestPoint, T19 TestPoint, T2 TestPoint, T20 TestPoint, T21 TestPoint, T22 TestPoint, T23 TestPoint, T24 TestPoint, T25 TestPoint, T26 TestPoint, T27 TestPoint, T28 TestPoint, T29 TestPoint, T3 TestPoint, T30 TestPoint, T4 TestPoint, T5 TestPoint, T6 TestPoint, T7 TestPoint, T8 TestPoint, T9 TestPoint

Commit message: Fix schematic and PCB connection mistake.
Connections:
- net Net-(J5-Pin_13) renamed /RESET_2
- J4 pad 3: GND -> /RESET_1
- J4 pad 4: Net-(J4-Pin_4) -> GND
- T3 pad 1: GND -> /RESET_1
- T4 pad 1: Net-(J4-Pin_4) -> GND
Routing:
- net Net-(J4-Pin_4): track 3.49 -> 0.00 mm
- net /RESET_1: track 0.00 -> 3.49 mm
Other:
- board text added: "WATER LEVEL SENSOR 0.6 F4INX 2026-04-20"
- board text removed: "WATER LEVEL SENSOR 0.5 F4INX 2026-03-28"
